File: PCB/Schematics/Memory.kicad_sch (KiCad schematic)
At the start: 10 parts, among them J8 Micro_SD_Card_Det1

Commit message: Add changes
Parts:
- J8: footprint SDSocket:microSD_HC_Molex_47219 -> Connector_Card:microSD_HC_Wuerth_693072010801
Changed lines of the file:
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@@
 			)
 		)
-		(property "Footprint" "SDSocket:microSD_HC_Molex_47219"
+		(property "Footprint" "Connector_Card:microSD_HC_Wuerth_693072010801"
 			(at 227.33 92.71 0)
 			(effects
