File: PCB/Schematics/POWER.kicad_sch (KiCad schematic)
At the start: 25 parts, among them J15 Power_In, Q1 IRF4905, U8 AMS1117-3.3, U9 TPS54202DDC

Commit message: Add changes
Parts:
- removed C37, C39: 100nF, Capacitor_SMD:C_0603_1608Metric, symbol Device:C
- removed C38: 10uF, Capacitor_SMD:C_0805_2012Metric, symbol Device:C
- removed C40, C41: 22uF, Capacitor_SMD:C_0805_2012Metric, symbol Device:C
- removed C42: 75pF, Capacitor_SMD:C_0603_1608Metric, symbol Device:C
- removed R29: 511K, Resistor_SMD:R_0603_1608Metric, symbol Device:R
- removed R30: 105K, Resistor_SMD:R_0603_1608Metric, symbol Device:R
- removed R31: 49.9R, Resistor_SMD:R_0603_1608Metric, symbol Device:R
- removed R32: 100K, Resistor_SMD:R_0603_1608Metric, symbol Device:R
- removed R33: 13.3K, Resistor_SMD:R_0603_1608Metric, symbol Device:R
- removed U9: TPS54202DDC, Package_TO_SOT_SMD:SOT-23-6, symbol Regulator_Switching:TPS54202DDC
- added C12, C18: 100nF, Capacitor_SMD:C_0603_1608Metric, symbol Device:C
- added C17: 10uF, Capacitor_SMD:C_0805_2012Metric, symbol Device:C
- added C19, C20: 22uF, Capacitor_SMD:C_0805_2012Metric, symbol Device:C
- added C21: 75pF, Capacitor_SMD:C_0603_1608Metric, symbol Device:C
- added R4: 511K, Resistor_SMD:R_0603_1608Metric, symbol Device:R
- added R5: 105K, Resistor_SMD:R_0603_1608Metric, symbol Device:R
- added R6: 49.9R, Resistor_SMD:R_0603_1608Metric, symbol Device:R
- added R7: 100K, Resistor_SMD:R_0603_1608Metric, symbol Device:R
- added R8: 13.3K, Resistor_SMD:R_0603_1608Metric, symbol Device:R
- added U7: TPS54202DDC, Package_TO_SOT_SMD:SOT-23-6, symbol Regulator_Switching:TPS54202DDC
- Q1: footprint Package_TO_SOT_THT:TO-220-3_Vertical -> IRF4905STRLPBF:TRANS_IRF3205S
Connections:
- net +24V: now also C12.1, C17.1, R4.1, U7.3 (VIN)
- net +5V: now also C19.1, C20.1, R6.1
- net GND: now also C12.2, C17.2, C19.2, C20.2, R5.2, R8.2, U7.1 (GND)
- net at L1.1: now also C18.2, U7.2 (SW)
- new net: C21.2, R7.2, R8.1, U7.4 (FB)
- new net: R4.2, R5.1, U7.5 (EN)
- new net: C18.1, U7.6 (BOOT)
- new net: C21.1, R6.2, R7.1
Other:
- moved on the sheet: C32, C33, C34, D1, D2, F1, J15, LED1, Q1, R28, R41, U8
